Commit message: Add STL meshes + URDF references + setup.py install

File: src/my_robot/urdf/robot_dh.urdf (robot description, URDF)
Before this commit: robot arm4dof, 6 links, 5 joints
Links:
- link link1: geometry collision box size=0.050 0.050 0.300; visual mesh filename=package://my_robot/meshes/Pieza1-0.17.stl scale=0.001 0.001 0.001
- link link2: geometry collision box size=0.400 0.040 0.040; visual mesh filename=package://my_robot/meshes/Pieza2-0.17.stl scale=0.001 0.001 0.001
- link link3: geometry collision box size=0.350 0.040 0.040; visual mesh filename=package://my_robot/meshes/Pieza6-0.17.stl scale=0.001 0.001 0.001
- link link4: geometry collision box size=0.200 0.040 0.040; visual mesh filename=package://my_robot/meshes/Pieza18-0.17.stl scale=0.001 0.001 0.001

Commit message: Feat:new

File: src/my_robot/urdf/robot_dh.urdf (robot description, URDF)
Before this commit: robot arm4dof, 6 links, 5 joints
Links:
- link link2: geometry collision box size=0.400 0.040 0.040; visual mesh filename=package://my_robot/meshes/Pieza2-0.17.stlas scale=0.001 0.001 0.001

Commit message: Feat:new

File: src/my_robot/urdf/robot_dh.urdf (robot description, URDF)
Before this commit: robot arm4dof, 6 links, 5 joints
Links:
- link link2: geometry collision box size=0.400 0.040 0.040; visual mesh filename=package://my_robot/meshes/Pieza2-0.17.stl scale=0.001 0.001 0.001
Joints:
- joint joint1: origin xyz=0.000000 0.000000 0.300000 rpy=1.570796 0.000000 1.570796 -> xyz=0 0 0.300000 rpy=-1.570796 0 1.570796
- joint joint2: origin xyz=0.400000 0.000000 0.000000 rpy=0.000000 0.000000 -1.570796 -> xyz=S 0 0 rpy=0 0 0
- joint joint3: origin xyz=0.350000 0.000000 0.000000 rpy=0.000000 0.000000 1.570796 -> xyz=0.350000 0 0 rpy=0 0 1.570796
- joint joint4: origin xyz=0.200000 0.000000 0.000000 rpy=1.570796 0.000000 0.000000 -> xyz=0.200000 0 0 rpy=1.570796 0 0

Commit message: Feat:new

File: src/my_robot/urdf/robot_dh.urdf (robot description, URDF)
Before this commit: robot arm4dof, 6 links, 5 joints
Links:
- link link2: geometry collision box size=0.400 0.040 0.040; visual mesh filename=package://my_robot/meshes/Pieza2-0.17.stlas scale=0.001 0.001 0.001
Joints:
- joint joint1: origin xyz=0 0 0.300000 rpy=-1.570796 0 1.570796 -> xyz=0.000000 0.000000 0.300000 rpy=1.570796 0.000000 1.570796
- joint joint2: origin xyz=S 0 0 rpy=0 0 0 -> xyz=0.400000 0.000000 0.000000 rpy=0.000000 0.000000 -1.570796
- joint joint3: origin xyz=0.350000 0 0 rpy=0 0 1.570796 -> xyz=0.350000 0.000000 0.000000 rpy=0.000000 0.000000 1.570796
- joint joint4: origin xyz=0.200000 0 0 rpy=1.570796 0 0 -> xyz=0.200000 0.000000 0.000000 rpy=1.570796 0.000000 0.000000
